File: Kicad/LIV2RIDE2K.kicad_pcb (KiCad board)
At the start: 2 copper layers, 56 parts, among them CN1 Zorro2, J1 JTAG, J2 LED, J3 LED, J4 Conn_02x22_Odd_Even, U1 AZ1117-3.3, U2 XC95144XL-TQ100, U3 74LVC245, U4 74LVC245, U5 MT48LC8M16A2P, U6 74HCT245, U7 74HCT245, U8 74HCT245, U9 SST39SF010, X1 50MHz

Commit message: A good start
Parts:
- removed C14, C15, C16, C17, C18, C19, C20, C21, C22, C23, C24, C25, C26: 0.1u, Capacitor_SMD:C_0603_1608Metric
- removed R7, R8, R9: 10K, Resistor_SMD:R_0603_1608Metric
- removed RN1: 10K, Resistor_SMD:R_Array_Convex_4x0603
- removed RN2, RN3, RN4, RN5: 22, Resistor_SMD:R_Array_Convex_4x0603
- removed U7, U8: 74HCT245, Package_SO:TSSOP-20_4.4x6.5mm_P0.65mm
- removed U9: SST39SF010, Package_SO:TSOP-I-32_11.8x8mm_P0.5mm
- removed X1: 50MHz, Oscillator:Oscillator_SMD_Abracon_ASE-4Pin_3.2x2.5mm_HandSoldering
- C13: value 10u -> 0.1u; footprint Capacitor_Tantalum_SMD:CP_EIA-3216-18_Kemet-A -> Capacitor_SMD:C_0603_1608Metric
- J3: value LED -> Conn_02x20_Odd_Even; footprint Connector_PinHeader_2.00mm:PinHeader_1x02_P2.00mm_Vertical -> Connector_IDC:IDC-Header_2x20_P2.54mm_Horizontal
- J4: value Conn_02x22_Odd_Even -> Conn_02x20_Odd_Even; footprint Connector_PinHeader_2.00mm:PinHeader_2x22_P2.00mm_Vertical -> Connector_IDC:IDC-Header_2x20_P2.54mm_Horizontal
- R2: value 33 -> 220
- R4: value 220 -> 10K
- U1: value AZ1117-3.3 -> LM1117-3.3; footprint Package_TO_SOT_SMD:SOT-89-3 -> Package_TO_SOT_SMD:SOT-223-3_TabPin2
- U2: value XC95144XL-TQ100 -> XC9572XL-VQ64; footprint Package_QFP:TQFP-100_14x14mm_P0.5mm -> Package_QFP:TQFP-64_10x10mm_P0.5mm
- U3, U4: value 74LVC245 -> 74HCT245
- U5: value MT48LC8M16A2P -> 74HCT245; footprint Package_SO:TSOP-II-54_22.2x10.16mm_P0.8mm -> Package_SO:TSSOP-20_4.4x6.5mm_P0.65mm
- U6: value 74HCT245 -> SST39SF010; footprint Package_SO:TSSOP-20_4.4x6.5mm_P0.65mm -> Package_SO:TSOP-I-32_11.8x8mm_P0.5mm
- moved C1 194.2 mm to (-118.6, 76.7)
- moved C11 194.2 mm to (-108.4, 70.7)
- moved C12 194.2 mm to (-100.2, 62.6)
- moved C2 194.2 mm to (-111.6, 67.8)
- moved C3 194.2 mm to (-93.1, 49.5)
- moved C4 194.2 mm to (-117.7, 73.9)
- moved C6 194.2 mm to (30.5, 39.5)
- moved F1 194.2 mm to (-85.5, 96.6)
- moved J2 194.2 mm to (-100.2, 57.3)
- moved R1 194.2 mm to (-112.4, 70.7)
- moved R2 194.2 mm to (-118.6, 79.2)
- moved R3 194.2 mm to (-88.5, 104.3)
- moved R4 194.2 mm to (-112.5, 104.3)
- moved R5 194.2 mm to (-112.5, 106.8)
- moved R6 194.2 mm to (-100.5, 104.3)
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Connections:
- C10 pad 1: +3.3V -> VCC
- C11 pad 1: +3.3V -> VCC
- C12 pad 1: +3.3V -> VCC
- C13 pad 1: +3.3V -> VCC
- CN1 pad 14: unconnected-(CN1-Pad14) -> /CPLD/~{C3}
- CN1 pad 15: unconnected-(CN1-Pad15) -> /CPLD/CDAC
- CN1 pad 16: unconnected-(CN1-Pad16) -> /CPLD/~{C1}
- CN1 pad 50: /CPLD/E -> unconnected-(CN1-Pad50)
- CN1 pad 93: /CPLD/DOE -> unconnected-(CN1-Pad93)
- F1 pad 2: Net-(F1-Pad2) -> unconnected-(F1-Pad2)
- J2 pad 1: /CPLD/FLASH_BANK -> Net-(J2-Pad1)
- J2 pad 2: VCC -> /IDE/~{LED}
- J3 pad 1: Net-(J3-Pad1) -> /IDE/B_~{RESET}
- J3 pad 2: /IDE/~{LED} -> GND
- J4 pad 29: /IDE/~{DMACK} -> unconnected-(J4-Pad29)
- J4 pad 37: /CPLD/~{IDE_CS1} -> /CPLD/~{IDE_CS2}
- J4 pad 38: /CPLD/~{IDE_CS2} -> unconnected-(J4-Pad38)
- R1 pad 1: GND -> /IDE/~{IDE_ACT}
- R1 pad 2: /CPLD/FLASH_BANK -> VCC
- R2 pad 1: Net-(R2-Pad1) -> VCC
- R2 pad 2: /CPLD/MEMCLK -> Net-(J2-Pad1)
- R3 pad 1: /IDE/~{IDE_ACT} -> /CPLD/IORDY
- R4 pad 1: VCC -> /IDE/~{IDE_IRQ}
- R4 pad 2: Net-(J3-Pad1) -> VCC
- R5 pad 1: /CPLD/IORDY -> /IDE/B_D15
- R6 pad 1: /IDE/~{DMACK} -> /IDE/B_D14
- U2 pad 1: /CPLD/~{IDE_ROMCS} -> /CPLD/~{DTACK}
- U2 pad 10: unconnected-(U2-Pad10) -> /CPLD/A16
- U2 pad 11: /CPLD/DOE -> /CPLD/~{BERR}
- U2 pad 12: /CPLD/~{SLAVE} -> /CPLD/A15
- U2 pad 13: /CPLD/~{CFGIN} -> /CPLD/A14
- U2 pad 14: /CPLD/~{CFGOUT} -> GND
- U2 pad 15: unconnected-(U2-Pad15) -> /CPLD/A13
- U2 pad 16: /CPLD/~{R_BUFOE} -> /CPLD/A12
- U2 pad 17: /CPLD/DQML -> /CPLD/A11
- U2 pad 18: /CPLD/RAM_~{W} -> /CPLD/A10
- U2 pad 19: /CPLD/DQMH -> /CPLD/A9
- U2 pad 2: /CPLD/~{IOWR} -> /CPLD/A23
- U2 pad 20: /CPLD/~{CAS} -> /CPLD/A1
- U2 pad 22: /CPLD/~{RAS} -> /CPLD/A8
- U2 pad 23: /CPLD/MEMCLK -> /CPLD/A2
- U2 pad 24: /CPLD/~{RAMCS} -> /CPLD/A7
- U2 pad 25: /CPLD/CKE -> /CPLD/A3
- U2 pad 27: /CPLD/BA0 -> /CPLD/A6
- U2 pad 28: /CPLD/MA11 -> /CPLD/TDI
- U2 pad 29: /CPLD/BA1 -> /CPLD/TMS
- U2 pad 3: /CPLD/~{IDE_CS2} -> +3.3V
- U2 pad 30: /CPLD/MA9 -> /CPLD/TCK
- U2 pad 31: GND -> /CPLD/A4
- U2 pad 32: /CPLD/MA10 -> /CPLD/A5
- U2 pad 33: /CPLD/MA8 -> /CPLD/~{IDE_ROMCS}
- U2 pad 34: /CPLD/MA0 -> /CPLD/~{OVR}
- U2 pad 35: /CPLD/MA7 -> /CPLD/CDAC
- U2 pad 36: /CPLD/MA1 -> /CPLD/~{C1}
- U2 pad 37: /CPLD/MA6 -> +3.3V
- U2 pad 38: +3.3V -> /CPLD/~{C3}
- U2 pad 39: /CPLD/MA2 -> /CPLD/~{CFGIN}
- U2 pad 4: /CPLD/~{IDE_CS1} -> /CPLD/A21
- U2 pad 40: /CPLD/MA5 -> /CPLD/~{CFGOUT}
- U2 pad 41: /CPLD/MA3 -> GND
- U2 pad 42: /CPLD/MA4 -> /CPLD/~{SLAVE}
- U2 pad 43: /CPLD/~{RAM_EN} -> unconnected-(U2-Pad43)
- U2 pad 44: GND -> unconnected-(U2-Pad44)
- U2 pad 45: /CPLD/TDI -> unconnected-(U2-Pad45)
- U2 pad 46: /CPLD/~{RANGER_EN} -> unconnected-(U2-Pad46)
- U2 pad 47: /CPLD/TMS -> unconnected-(U2-Pad47)
- U2 pad 48: /CPLD/TCK -> unconnected-(U2-Pad48)
- U2 pad 49: /CPLD/~{IDE_EN} -> unconnected-(U2-Pad49)
- U2 pad 5: +3.3V -> /CPLD/A22
- U2 pad 51: +3.3V -> unconnected-(U2-Pad51)
- U2 pad 52: /CPLD/~{UDS} -> /CPLD/D12
- U2 pad 53: /CPLD/~{AS} -> /CPLD/TDO
- U2 pad 54: /CPLD/R~{W} -> GND
- U2 pad 55: /CPLD/~{LDS} -> +3.3V
- U2 pad 56: /CPLD/~{DTACK} -> /CPLD/D13
- U2 pad 57: +3.3V -> /CPLD/D14
- U2 pad 58: /CPLD/D13 -> /CPLD/D15
- U2 pad 59: /CPLD/D12 -> /CPLD/~{I_BUFOE}
- U2 pad 6: /CPLD/IORDY -> /CPLD/A20
- U2 pad 60: /CPLD/D15 -> /CPLD/~{AS}
- U2 pad 61: /CPLD/D14 -> /CPLD/~{UDS}
- U2 pad 62: GND -> /CPLD/~{LDS}
- U2 pad 63: /CPLD/A20 -> /CPLD/R~{W}
- U2 pad 64: /CPLD/A21 -> /CPLD/~{RST}
- U2 pad 7: /CPLD/~{I_BUFOE} -> /CPLD/A19
- U2 pad 8: unconnected-(U2-Pad8) -> /CPLD/A18
- U2 pad 9: unconnected-(U2-Pad9) -> /CPLD/A17
- U3 pad 13: /CPLD/D7 -> /CPLD/D4
- U3 pad 14: /CPLD/D4 -> /CPLD/D7
- U3 pad 16: /CPLD/D2 -> /CPLD/D8
- U3 pad 17: /CPLD/D1 -> /CPLD/D2
- U3 pad 18: /CPLD/D0 -> /CPLD/D9
- U3 pad 19: /CPLD/~{R_BUFOE} -> /CPLD/~{I_BUFOE}
- U3 pad 2: Net-(RN2-Pad4) -> /IDE/B_D9
- U3 pad 20: +3.3V -> VCC
- U3 pad 3: Net-(RN2-Pad3) -> /IDE/B_D2
- U3 pad 4: Net-(RN2-Pad2) -> /IDE/B_D8
- U3 pad 5: Net-(RN2-Pad1) -> /IDE/B_D3
- U3 pad 6: Net-(RN3-Pad4) -> /IDE/B_D7
- U3 pad 7: Net-(RN3-Pad3) -> /IDE/B_D4
- U3 pad 8: Net-(RN3-Pad2) -> /IDE/B_D6
- U3 pad 9: Net-(RN3-Pad1) -> /IDE/B_D5
- U4 pad 11: /CPLD/D15 -> /CPLD/D1
- U4 pad 12: /CPLD/D14 -> /CPLD/D10
- U4 pad 13: /CPLD/D13 -> /CPLD/D0
- U4 pad 14: /CPLD/D12 -> /CPLD/D11
- U4 pad 15: /CPLD/D11 -> /CPLD/D12
- U4 pad 16: /CPLD/D10 -> /CPLD/D13
- U4 pad 17: /CPLD/D9 -> /CPLD/D14
- U4 pad 18: /CPLD/D8 -> /CPLD/D15
- U4 pad 19: /CPLD/~{R_BUFOE} -> /CPLD/~{I_BUFOE}
- U4 pad 2: Net-(RN4-Pad4) -> /IDE/B_D15
- U4 pad 20: +3.3V -> VCC
- U4 pad 3: Net-(RN4-Pad3) -> /IDE/B_D14
- U4 pad 4: Net-(RN4-Pad2) -> /IDE/B_D13
- U4 pad 5: Net-(RN4-Pad1) -> /IDE/B_D12
- U4 pad 6: Net-(RN5-Pad4) -> /IDE/B_D11
- U4 pad 7: Net-(RN5-Pad3) -> /IDE/B_D0
- U4 pad 8: Net-(RN5-Pad2) -> /IDE/B_D10
- U4 pad 9: Net-(RN5-Pad1) -> /IDE/B_D1
- U5 pad 1: +3.3V -> GND
- U5 pad 10: /RAM/R_D5 -> GND
- U5 pad 11: /RAM/R_D6 -> /CPLD/~{RST}
- U5 pad 13: /RAM/R_D7 -> GND
- U5 pad 14: +3.3V -> /CPLD/A11
- U5 pad 15: /CPLD/DQML -> /CPLD/A10
- U5 pad 16: /CPLD/RAM_~{W} -> /CPLD/A9
- U5 pad 17: /CPLD/~{CAS} -> /IDE/~{IDE_ACT}
- U5 pad 18: /CPLD/~{RAS} -> /IDE/~{IDE_ACT}
- U5 pad 19: /CPLD/~{RAMCS} -> GND
- U5 pad 2: /RAM/R_D0 -> /IDE/~{LED}
- U5 pad 20: /CPLD/BA0 -> VCC
- U5 pad 3: +3.3V -> /IDE/~{LED}
- U5 pad 4: /RAM/R_D1 -> /IDE/I_A0
- U5 pad 5: /RAM/R_D2 -> /IDE/I_A1
- U5 pad 6: GND -> /IDE/I_A2
- U5 pad 7: /RAM/R_D3 -> unconnected-(U5-Pad7)
- U5 pad 8: /RAM/R_D4 -> unconnected-(U5-Pad8)
- U5 pad 9: +3.3V -> /IDE/B_~{RESET}
- U6 pad 1: /CPLD/R~{W} -> /CPLD/A12
- U6 pad 11: /CPLD/D11 -> GND
- U6 pad 12: /CPLD/D4 -> /CPLD/A13
- U6 pad 13: /CPLD/D10 -> /CPLD/A8
- U6 pad 14: /CPLD/D5 -> /CPLD/A7
- U6 pad 15: /CPLD/D9 -> /CPLD/A6
- U6 pad 16: /CPLD/D6 -> /CPLD/A5
- U6 pad 17: /CPLD/D8 -> /CPLD/A4
- U6 pad 18: /CPLD/D7 -> /CPLD/A3
- U6 pad 19: /CPLD/~{I_BUFOE} -> /CPLD/A2
- U6 pad 2: /IDE/B_D7 -> /CPLD/A10
- U6 pad 20: VCC -> /CPLD/A1
- U6 pad 3: /IDE/B_D8 -> /CPLD/A9
- U6 pad 4: /IDE/B_D6 -> /CPLD/A14
- U6 pad 5: /IDE/B_D9 -> /CPLD/A15
- U6 pad 6: /IDE/B_D5 -> GND
- U6 pad 7: /IDE/B_D10 -> /CPLD/~{IOWR}
- U6 pad 8: /IDE/B_D4 -> VCC
- U6 pad 9: /IDE/B_D11 -> GND
Routing:
- net /IDE/B_D15: track 0.00 -> 121.1 mm, vias 0 -> 2
- net /IDE/B_D14: track 0.00 -> 116.1 mm, vias 0 -> 2
- net /IDE/B_D13: track 0.00 -> 113.0 mm, vias 0 -> 2
- net /IDE/B_D1: track 0.00 -> 112.1 mm, vias 0 -> 1
- net /IDE/B_D12: track 0.00 -> 107.5 mm, vias 0 -> 2
- net /IDE/B_D11: track 0.00 -> 106.0 mm, vias 0 -> 2
- net /IDE/B_D2: track 0.00 -> 103.7 mm, vias 0 -> 1
- net /IDE/B_D3: track 0.00 -> 99.6 mm, vias 0 -> 1
- net /IDE/B_D10: track 0.00 -> 96.8 mm, vias 0 -> 1
- net /IDE/B_D4: track 0.00 -> 96.3 mm, vias 0 -> 1
- net /IDE/B_D7: track 0.00 -> 92.9 mm
- net /IDE/B_D6: track 0.00 -> 92.7 mm
- net /IDE/B_D5: track 0.00 -> 92.5 mm
- net /IDE/B_D9: track 0.00 -> 90.1 mm, vias 0 -> 1
- net /IDE/B_D8: track 0.00 -> 89.7 mm
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Other:
- board outline added: 129.5 x 50.1 mm
- board text added: "DON'T FORGET TO ADD KEY PWR!!!"
