File: Kicad/LIV2RIDE2K.kicad_sch (KiCad schematic)
At the start: 0 parts

Commit message: A good start
Other:
- removed sheet RAM
- sheet CPLD ports: added none; removed BA0, BA1, CKE, DQMH, DQML, MEMCLK, RAM_~{W}, ~{CAS}, ~{RAMCS}, ~{RAS}, ~{R_BUFOE}
